File: greymechaarmy_v2/hardware/greybadge_pcb/greybadge_pcb.kicad_sch (KiCad schematic)
At the start: 86 parts, among them J1 Conn_02x05_Row_Letter_First, J2 Conn_02x05_Row_Letter_First, J3 Conn_02x05_Row_Letter_First, J4 JST PH S2B, Q1 2N7002, SW1 SW_Push, SW2 SW_Push, SW3 SW_Push, SW4 SW_Push, SW5 SW_Push, SW6 SW_Push, SW7 SW_Push, SW8 SW_SPDT, U10 AMS1117-3.3, U2 TLV73311PDBV, U3 TLV73325PDBV, U4 GC9A01_IPS_display, U5 BQ24075

Commit message: feat: add additional pmod header with differential lines
Parts:
- added J6: Conn_02x05_Row_Letter_First, Connector_PinSocket_2.54mm:PinSocket_2x06_P2.54mm_Vertical_SMD, symbol Connector_Generic:Conn_02x06_Odd_Even
Connections:
- net +3V3: now also J6.1 (Pin_1), J6.2 (Pin_2)
- net GND: now also J6.3 (Pin_3), J6.4 (Pin_4)
- new net D1: J6.11 (Pin_11)
- new net E1: J6.7 (Pin_7)
- new net E2: J6.9 (Pin_9)
- new net F2: J6.5 (Pin_5)
- new net PMOD1+: J6.10 (Pin_10)
- new net PMOD1-: J6.12 (Pin_12)
- new net PMOD2+: J6.6 (Pin_6)
- new net PMOD2-: J6.8 (Pin_8)
Other:
- note added: "FPGA (bottom)"
- note added: "FPGA (top)"
- note removed: "FPGA"
- moved on the sheet: J3, JP1, JP2, JP3, JP4, JP5
